File: Night light PCB.kicad_pcb (KiCad board)
At the start: 4 copper layers, 242.1 x 170 mm, 152 parts, among them IC1 NRF24L01P-R, IC2 TLV3012AIDBVTG4, IC3 BISS0001, IC4 STM32G031K8T6TR, IC5 NRF24L01P-R, J1 Battery, J2 Conn_ARM_SWD_TagConnect_TC2030, J3 Conn_ARM_SWD_TagConnect_TC2030, J4 Conn_01x01_Pin, J5 Conn_01x01_Pin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

Commit message: Update
Parts:
- removed FL1: RN112-0.8-02-10M, 10MH CHOKE:RN112080210M
- removed REF** (x5): MountingHole_3.2mm_M3_ISO7380, MountingHole:MountingHole_3.2mm_M3_ISO7380
- removed Y3: Crystal, Crystal:Crystal_SMD_5032-2Pin_5.0x3.2mm
- removed mouse-bite-2mm-4mm (x9): VAL**, mouse bite:mouse-bite-2mm-4mm
- added D1: LED, LED_SMD:LED_0402_1005Metric, F.Cu at (258.7, 89.3)
- added FL2: UU9.8-10MH, 10MH CHOKE:UU9810MH, F.Cu at (70.8, 123.4)
- added H1: MountingHole, MountingHole:MountingHole_3.2mm_M3, F.Cu at (268.9, 112.7)
- added H2: MountingHole, MountingHole:MountingHole_3.2mm_M3, F.Cu at (215.0, 79.0)
- added H3: MountingHole, MountingHole:MountingHole_3.2mm_M3, F.Cu at (116.2, 154.6)
- added H4: MountingHole, MountingHole:MountingHole_3.2mm_M3, F.Cu at (101.5, 39.8)
- added H5: MountingHole, MountingHole:MountingHole_3.2mm_M3, F.Cu at (191.9, 97.7)
- added R52: 330r, Resistor_SMD:R_0402_1005Metric, F.Cu at (258.7, 90.4)
- added TP1: LDO_IN, TestPoint:TestPoint_Pad_D4.0mm, F.Cu at (95.1, 37.9)
- added U10: mouse bite, mouse bite:mouse-bite-2mm-4mm, F.Cu at (54.0, 94.7)
- added U11: mouse bite, mouse bite:mouse-bite-2mm-4mm, F.Cu at (130.5, 18.8)
- added U12: mouse bite, mouse bite:mouse-bite-2mm-4mm, F.Cu at (206.0, 93.9)
- added U13: mouse bite, mouse bite:mouse-bite-2mm-4mm, F.Cu at (242.0, 69.7)
- added U3: mouse bite, mouse bite:mouse-bite-2mm-4mm, F.Cu at (242.0, 121.9)
- added U5: mouse bite, mouse bite:mouse-bite-2mm-4mm, F.Cu at (242.0, 170.1)
- added U7: mouse bite, mouse bite:mouse-bite-2mm-4mm, F.Cu at (242.0, 18.7)
- added U8: mouse bite, mouse bite:mouse-bite-2mm-4mm, F.Cu at (130.4, 170.8)
- added U9: mouse bite, mouse bite:mouse-bite-2mm-4mm, F.Cu at (278.1, 93.8)
- added Y1: crystal, crystal:X322516MOB4SI, F.Cu at (254.7, 88.9)
- C38: value 563pf -> 56nf
- F1: value SF-3812TL100T-2 -> JFC2410-1100TS
- R19: value 10k -> 120k
- R41, R42, R43, R44, R45, R46: value 18 -> 33R; footprint Resistor_SMD:R_0402_1005Metric -> Resistor_SMD:R_0805_2012Metric
- Y2: value Crystal -> crystal; footprint Crystal:Crystal_SMD_5032-2Pin_5.0x3.2mm -> crystal:X322516MOB4SI
- moved C23 2.00 mm to (183.0, 85.2)
- moved Y2 1.31 mm to (185.0, 81.8), turned to -130 degrees
- moved C49 1.28 mm to (258.5, 88.1)
- moved C25 0.84 mm to (187.1, 78.5)
- moved R41 0.26 mm to (70.5, 103.8)
- moved R43 0.21 mm to (151.9, 38.7)
- moved R45 0.16 mm to (108.1, 150.7)
Connections:
- U2 pad 5: unconnected-(U2-PA7-Pad5) -> Net-(U2-PA7)
- Y2 pad 1: Net-(IC1-XC2) -> Net-(IC1-XC1)
- Y2 pad 2: Net-(IC1-XC1) -> GND
Routing:
- net Net-(U2-PA7): track 0.00 -> 27.4 mm, vias 0 -> 2
- net Net-(C4-Pad1): track 21.2 -> 34.3 mm
- net Net-(PS1-AC/N): track 16.1 -> 24.3 mm
- net /LDO_IN: track 30.1 -> 38.0 mm, vias 0 -> 2
- net GND: track 86.4 -> 91.7 mm, vias 37 -> 54
- net GNDREF: track 14.4 -> 19.6 mm, vias 11 -> 27
- net Net-(PS1-AC/L): track 21.2 -> 16.3 mm
- net /3V3: track 42.6 -> 46.6 mm
- net /N: track 41.2 -> 44.5 mm
- net Net-(IC1-XC2): track 6.64 -> 9.65 mm
- net Net-(IC5-XC2): track 6.76 -> 9.14 mm
- net Net-(D1-A): track 0.00 -> 1.15 mm
- net Net-(IC1-XC1): track 7.01 -> 7.90 mm
Other:
- board text added: "+"
- board text added: "-"
- board text added: "D"
- board text added: "G"
- board text added: "L"
- board text added: "N"
- board text added: "RF / Impedance Note Controlled impedance trace(s): 50 Ω single-ended Applies to: antenna feedline only (50ohm & 50ohm_) Stackup: standard 4-layer FR4 (1.6062 mm, 1 oz copper) Reference plane: solid continuous ground plane on inner layer 1 Tolerance: ±10% impedance tolerance Routing requirement: no discontinuities, maintain constant trace width and clearance per calculated geometry"
- board text added: "S"
- board text added: "layer {dblquote}F.Silkscreen{dblquote} type {dblquote}Top Silk Screen{dblquote} Color {dblquote}Not specified{dblquote} Material {dblquote}Not specified{dblquote} layer {dblquote}F.Paste{dblquote} type {dblquote}Top Solder Paste{dblquote} layer {dblquote}F.Mask{dblquote} type {dblquote}Top Solder Mask{dblquote} Color {dblquote}Not specified{dblquote} Thickness 0.01 mm Material {dblquote}Not speci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"
- board text removed: "RF / Impedance Note (recommended) Controlled impedance trace(s): 50 Ω single-ended Applies to: antenna feedline only (50ohm & 50ohm_) Stackup: standard 4-layer FR4 (1.6062 mm, 1 oz copper) Reference plane: solid continuous ground plane on inner layer 1 Tolerance: ±10% impedance tolerance (typical PCB fab standard) Routing requirement: no discontinuities, maintain constant trace width and clearanc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"
- board text removed: "layer "F.Silkscreen" type "Top Silk Screen" Color "Not specified" Material "Not specified" layer "F.Paste" type "Top Solder Paste" layer "F.Mask" type "Top Solder Mask" Color "Not specified" Thickness 0.01 mm Material "Not specified" EpsilonR 3.3 LossTg 0 layer "F.Cu" type "copper" Thickness 0.035 mm layer "Dielectric 1" type "prepreg" sublayer "1/1" Color "Not specified" Thickness 0.2104 mm Mate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"
