File: Night light PCB.kicad_sch (KiCad schematic)
At the start: 124 parts, among them IC1 STM32G031K8T6TR, IC2 BISS0001, J1 Battery, J2 Conn_ARM_SWD_TagConnect_TC2030, J3 Conn_ARM_SWD_TagConnect_TC2030, Q1 AO3400A, Q2 AO3407A, U1 BQ24074RGT, U2 TLV75533PDBV, U3 nRF24L01P, U4 PIS-209S, U5 ATtiny1616-S, U6 nRF24L01P, U7 BC2AAPC, Y1 Crystal, Y2 Crystal

Commit message: update
Parts:
- removed C34: 100nf, Capacitor_SMD:C_0402_1005Metric, symbol Device:C
- removed C38: 33nf, Capacitor_SMD:C_0402_1005Metric, symbol Device:C
- removed C39, C40: 22pf, Capacitor_SMD:C_0402_1005Metric, symbol Device:C
- removed C41: 1nf, Capacitor_SMD:C_0805_2012Metric, symbol Device:C
- removed C42: 10nf, Capacitor_SMD:C_0805_2012Metric, symbol Device:C
- removed C43: 100nf, Capacitor_SMD:C_0805_2012Metric, symbol Device:C
- removed C44: 1.5pf, Capacitor_SMD:C_0402_1005Metric, symbol Device:C
- removed C45: 4.7pf, Capacitor_SMD:C_0402_1005Metric, symbol Device:C
- removed C46: 1pf, Capacitor_SMD:C_0402_1005Metric, symbol Device:C
- removed D1, D2: LED, LED_SMD:LED_0402_1005Metric, symbol Device:LED
- removed D3, D4, D5, D6, D7, D8: LED, symbol Device:LED
- removed F1: Fuse, symbol Device:Fuse
- removed FL1: RN112-0.8-02-10M, RN112080210M, symbol 10mh choke:RN112-0.8-02-10M
- removed IC1: STM32G031K8T6TR, QFP80P900X900X160-32N, symbol STM32:STM32G031K8T6TR
- removed JP1: SolderJumper_3_Open, Jumper:SolderJumper-3_P2.0mm_Open_TrianglePad1.0x1.5mm, symbol Jumper:SolderJumper_3_Open
- removed JP2: SolderJumper_3_Open, symbol Jumper:SolderJumper_3_Open
- removed L4: 8.2nH, Inductor_SMD:L_0402_1005Metric, symbol Device:L
- removed L5: 3.9nH, Inductor_SMD:L_0402_1005Metric, symbol Device:L
- removed L6: 2.7nH, Inductor_SMD:L_0402_1005Metric, symbol Device:L
- removed R1, R2: 1.5k, Resistor_SMD:R_0402_1005Metric, symbol Device:R
- removed R34, R35: 100k, Resistor_SMD:R_0402_1005Metric, symbol Device:R
- removed R38: 22k, Resistor_SMD:R_0402_1005Metric, symbol Device:R
- removed R39: ~, Resistor_SMD:R_0402_1005Metric, symbol Device:R
- removed U3, U6: nRF24L01P, Package_DFN_QFN:QFN-20-1EP_4x4mm_P0.5mm_EP2.5x2.5mm, symbol RF:nRF24L01P
- removed U7: BC2AAPC, BC2AAPC, symbol AA bat:BC2AAPC
- removed Y1, Y2: Crystal, Crystal:Crystal_SMD_5032-2Pin_5.0x3.2mm, symbol Device:Crystal
- added BT1: Battery, Battery:BatteryHolder_Keystone_2468_2xAAA, symbol Device:Battery
- added C48, C49: 22pf, Capacitor_SMD:C_0402_1005Metric, symbol Device:C
- added C50: 1nf, Capacitor_SMD:C_0402_1005Metric, symbol Device:C
- added C51: 10nf, Capacitor_SMD:C_0402_1005Metric, symbol Device:C
- added C52: 2.2nf, Capacitor_SMD:C_0402_1005Metric, symbol Device:C
- added C53: 100nf, Capacitor_SMD:C_0402_1005Metric, symbol Device:C
- added C54: 4.7pf, Capacitor_SMD:C_0402_1005Metric, symbol Device:C
- added C55: 1.5pf, Capacitor_SMD:C_0402_1005Metric, symbol Device:C
- added C56: 1pf, Capacitor_SMD:C_0402_1005Metric, symbol Device:C
- added F1: JFC2410-1100TS, FUSE:FUSC10131X330N, symbol FUSE:SF-3812TL100T-2
- added FL2: UU9.8-10MH, UU9810MH, symbol 10mh choke:UU9.8-10MH
- added IC1, IC5: NRF24L01P-R, nRF24L01P:QFN50P400X400X95-21N-D, symbol nRF24L01P:NRF24L01P-R
- added IC2: TLV3012AIDBVTG4, TLV3012:SOT95P280X145-6N, symbol TLV3012:TLV3012AIDBVTG4
- added IC4: STM32G031K8T6TR, STM32:QFP80P900X900X160-32N, symbol STM32:STM32G031K8T6TR
- added J4, J5: Conn_01x01_Pin, TestPoint:TestPoint_Keystone_5010-5014_Multipurpose, symbol Connector:Conn_01x01_Pin
- added L7: 8.2nH, Inductor_SMD:L_0402_1005Metric, symbol Device:L
- added L8: 2.7nH, Inductor_SMD:L_0402_1005Metric, symbol Device:L
- added L9: 3.9nH, Inductor_SMD:L_0402_1005Metric, symbol Device:L
- added LED1, LED2, LED3, LED4, LED5, LED6: SPMWH1228MD5WATUVK, LED:SPMWH1228MD5WATUVK, symbol LED:SPMWH1228MD5WATUVK
- added Q2: AO3400A, Package_TO_SOT_SMD:SOT-23, symbol Transistor_FET:AO3400A
- added Q3: AO3407A, PMOS A03407:SOT95P280X125-3N, symbol PMOS-AO3407A:AO3407A
- added R11, R16, R17, R18, R22, R48, R49, R5, R50, R51, R9: 10k, Resistor_SMD:R_0402_1005Metric, symbol Device:R
- added R12: 174k, Resistor_SMD:R_0402_1005Metric, symbol Device:R
- added R13: 100k, Resistor_SMD:R_0402_1005Metric, symbol Device:R
- added R14, R47: 1M, Resistor_SMD:R_0402_1005Metric, symbol Device:R
- added R15: 100r, Resistor_SMD:R_0402_1005Metric, symbol Device:R
- added R6: 22k, Resistor_SMD:R_0402_1005Metric, symbol Device:R
- added S1, S2, S3: 1301.9314.24, Switch:1301931424, symbol SWITCH:1301.9314.24
- added Y1, Y2: crystal, X322516MOB4SI, symbol crystal:X322516MOB4SI
- C1: renamed from C4; JLCPCB PART # (none) -> C29266
- C10: renamed from C2; JLCPCB PART # (none) -> C125977
- C11: renamed from C3; JLCPCB PART # (none) -> C98192
- C12: renamed from C6; JLCPCB PART # (none) -> C28323
- C14: renamed from C7; JLCPCB PART # (none) -> C95841
- C16: renamed from C14; JLCPCB PART # (none) -> C106862
- C19: renamed from C28; JLCPCB PART # (none) -> C2918502
- C2: renamed from C35; JLCPCB PART # (none) -> C94121
- C21: renamed from C26; JLCPCB PART # (none) -> C5440143
- C22: renamed from C21; JLCPCB PART # (none) -> C18185763
- C23: renamed from C15; JLCPCB PART # (none) -> C277482
- C25: renamed from C16; JLCPCB PART # (none) -> C277482
- C26: renamed from C29; JLCPCB PART # (none) -> C5440143
- C28: renamed from C8; footprint Capacitor_SMD:C_0805_2012Metric -> Capacitor_SMD:C_0402_1005Metric; JLCPCB PART # (none) -> C76947
- C3: renamed from C12; JLCPCB PART # (none) -> C49678
- C30: renamed from C22; JLCPCB PART # (none) -> C36911349
- C31: renamed from C9; footprint Capacitor_SMD:C_0805_2012Metric -> Capacitor_SMD:C_0402_1005Metric; JLCPCB PART # (none) -> C15195
- C34: renamed from C23; JLCPCB PART # (none) -> C701296
- C35: renamed from C24; JLCPCB PART # (none) -> C5440143
- C36: renamed from C13; footprint Capacitor_SMD:C_0805_2012Metric -> Capacitor_SMD:C_0402_1005Metric; JLCPCB PART # (none) -> C60474
- C37: renamed from C27; JLCPCB PART # (none) -> C327009
- C38: renamed from C25; value 563pf -> 56nf; JLCPCB PART # (none) -> C36911349
- C39: renamed from C19; JLCPCB PART # (none) -> C1552
- C4: renamed from C1; JLCPCB PART # (none) -> C46638858
- C40: renamed from C17; JLCPCB PART # (none) -> C1569
- C41: renamed from C30; JLCPCB PART # (none) -> C5440143
- C42: renamed from C20; JLCPCB PART # (none) -> C710646
- C43: renamed from C18; JLCPCB PART # (none) -> C2987940
- C44: renamed from C31; JLCPCB PART # (none) -> C701296
- C45: renamed from C33; JLCPCB PART # (none) -> C701296
- C46: renamed from C32; JLCPCB PART # (none) -> C36911349
- C47: value 2.2nf -> 33nf; JLCPCB PART # (none) -> C106862
- C5: renamed from C11; JLCPCB PART # (none) -> C98192
- C6: renamed from C36; JLCPCB PART # (none) -> C49678
- C7: renamed from C10; JLCPCB PART # (none) -> C49678
- C8: renamed from C37; JLCPCB PART # (none) -> C98192
- C9: renamed from C5; JLCPCB PART # (none) -> C98192
- IC3: renamed from IC2; footprint SOIC127P600X160-16N -> BISS0001:SOIC127P600X160-16N; JLCPCB PART # (none) -> C18164474
- J1: footprint Connector_JST:JST_XA_S02B-XASK-1_1x02_P2.50mm_Horizontal -> Connector_JST:JST_EH_B2B-EH-A_1x02_P2.50mm_Vertical; now not fitted
- J2: renamed from J3; now not fitted
- J3: renamed from J2; now not fitted
- L4: renamed from L1; JLCPCB PART # (none) -> C84404
- L5: renamed from L2; JLCPCB PART # (none) -> C5452416
- L6: renamed from L3; JLCPCB PART # (none) -> C77108
- PS1: JLCPCB PART # (none) -> C209907
- Q1: renamed from Q2; footprint SOT95P280X125-3N -> PMOS A03407:SOT95P280X125-3N; JLCPCB PART # (none) -> C15155; now not fitted
- Q4: renamed from Q1; JLCPCB PART # (none) -> C20917; now not fitted
- R1: renamed from R4; JLCPCB PART # (none) -> C138017
- R10: renamed from R40; JLCPCB PART # (none) -> C60491
- R19: renamed from R25; value 10k -> 120k; JLCPCB PART # (none) -> C60490
- R2: renamed from R36; JLCPCB PART # (none) -> C60490
- R20: renamed from R24; JLCPCB PART # (none) -> C125627
- R21: renamed from R6; JLCPCB PART # (none) -> C82868
- R23: renamed from R17; JLCPCB PART # (none) -> C138044
- R24: renamed from R10; JLCPCB PART # (none) -> C138044
- R25: renamed from R16; JLCPCB PART # (none) -> C138044
- R26: renamed from R8; value ~ -> 1M; JLCPCB PART # (none) -> C138033
- R27: renamed from R15; JLCPCB PART # (none) -> C137946
- R28: renamed from R9; JLCPCB PART # (none) -> C138044
- R29: renamed from R14; JLCPCB PART # (none) -> C60491
- R3: renamed from R5; JLCPCB PART # (none) -> C163481
- R30: renamed from R11; JLCPCB PART # (none) -> C138044
- R31: renamed from R13; JLCPCB PART # (none) -> C203143
- R32: renamed from R12; JLCPCB PART # (none) -> C138033
- R33: renamed from R18; JLCPCB PART # (none) -> C138033
- R34: renamed from R19; JLCPCB PART # (none) -> C482174
- R35: renamed from R20; JLCPCB PART # (none) -> C137946
- R36: renamed from R23; JLCPCB PART # (none) -> C25760
- R37: renamed from R22; JLCPCB PART # (none) -> C3013173
- R38: renamed from R32; JLCPCB PART # (none) -> C106232
- R39: renamed from R21; JLCPCB PART # (none) -> C137976
- R4: renamed from R3; now not fitted
- R40: renamed from R33; value 100k -> 10k; JLCPCB PART # (none) -> C60490
- R41: renamed from R26; value 18 -> 33R; JLCPCB PART # (none) -> C138002
- R42: renamed from R27; value 18 -> 33R; JLCPCB PART # (none) -> C138002
- R43: renamed from R28; value 18 -> 33R; JLCPCB PART # (none) -> C138002
- R44: renamed from R29; value 18 -> 33R; JLCPCB PART # (none) -> C138002
- R45: renamed from R30; value 18 -> 33R; JLCPCB PART # (none) -> C138002
- R46: renamed from R31; value 18 -> 33R; JLCPCB PART # (none) -> C138002
- R7: renamed from R37; JLCPCB PART # (none) -> C105871
- R8: renamed from R7; JLCPCB PART # (none) -> C60490
- RV1: JLCPCB PART # (none) -> C2839517
- U1: JLCPCB PART # (none) -> C54313; now not fitted
- U2: renamed from U5; JLCPCB PART # (none) -> C614136; now not fitted
- U4: renamed from U2; JLCPCB PART # (none) -> C404027; now not fitted
- U6: renamed from U4; footprint PIS209S -> PIS209S:PIS209S; now not fitted
- VR1: footprint PVG3A103C01R00 -> 10k trimmer:PVG3A103C01R00; JLCPCB PART # (none) -> C780220
Connections:
- net +3.3V: now also BT1.1 (+), C50.1, C51.1, C53.1, IC5.15 (VDD_2), IC5.18 (VDD_3), IC5.7 (VDD_1), R11.1, R17.1, R18.2, R48.1, R9.1
- net 3V3: now also IC3.1 (A), R41.2, R42.2, R43.2, R44.2, R45.2, R46.2, IC1.15 (VDD_2), IC1.18 (VDD_3), IC1.7 (VDD_1), IC4.4 (VDD/VDDA), R50.2, R51.1; no longer R41.1, R42.1, R43.1, R44.1, R45.1, R46.1
- net CE: now also IC1.1 (CE), IC4.15 (PB0), R49.2
- net CE_: now also U2.13 (PC1), IC5.1 (CE), R22.2; no longer U2.3 (PA5)
- net CSN: now also IC1.2 (CSN), IC4.10 (PA3), R50.1
- net CSN_: now also U2.12 (PC0), IC5.2 (CSN), R18.1; no longer U2.2 (PA4)
- net GND: now also C1.2, U1.17 (VSS), U1.8 (VSS), IC1.14 (VSS_2), IC1.17 (VSS_3), IC1.20 (VSS_4), IC1.8 (VSS_1), IC2.2 (V-), IC4.5 (VSS/VSSA), Q2.2 (S), R13.1, R16.2, R49.1, Y2.2 (GND_1), Y2.4 (GND_2)
- net GNDREF: now also BT1.2 (-), C48.2, C49.2, C50.2, C51.2, C52.2, C53.2, C54.2, C56.2, IC5.14 (VSS_2), IC5.17 (VSS_3), IC5.20 (VSS_4), IC5.8 (VSS_1), R22.1, R6.2, S1.3 (COM_1), S1.4 (COM_2), S2.3 (COM_1), S2.4 (COM_2), S3.3 (COM_1), S3.4 (COM_2), Y1.2 (GND_1), Y1.4 (GND_2)
- net IRQ: now also IC1.6 (IRQ), IC4.16 (PB1), R51.2
- net IRQ_: now also U2.14 (PC2), IC5.6 (IRQ), R48.2; no longer U2.4 (PA6)
- net L: now also F1.1, J4.1 (Pin_1)
- net Led-drive: now also IC4.19 (PA9)
- net Light-sense: now also IC4.8 (PA1)
- net MISO_: now also IC5.5 (MISO)
- net MOSI_: now also IC5.4 (MOSI)
- net N: now also FL2.4, J5.1 (Pin_1)
- net NRST: now also IC4.6 (PF2-NRST)
- net PIR-VO: now also IC4.18 (PA8)
- net SCK_: now also IC5.3 (SCK)
- net SPI1_MISO: now also IC1.4 (MOSI), IC4.13 (PA6)
- net SPI1_MOSI: now also IC1.5 (MISO), IC4.14 (PA7)
- net SPI1_SCK: now also IC1.3 (SCK), IC4.12 (PA5)
- net SWCLK: now also IC4.25 (PA14-BOOT0)
- net SWDIO: now also IC4.24 (PA13)
- net SYS: now also Q3.2 (S), R5.2; no longer C12.1, U4.1 (IN), U4.3 (EN)
- net at PS1.2 (AC/N): now also FL2.3
- net at C4.1, RV1.1: now also F1.2, FL2.1
- net at PS1.1 (AC/L): now also FL2.2
- net at R21.1: now also IC1.16 (IREF)
- net at Q4.3 (D): now also LED1.1 (K), LED2.1 (K), LED3.1 (K), LED4.1 (K), LED5.1 (K), LED6.1 (K)
- net at C23.1, R26.2: now also IC1.9 (XC2), Y2.3 (CRYSTAL_2)
- net at C25.1, R26.1: now also IC1.10 (XC1), Y2.1 (CRYSTAL_1)
- net at C40.1, C43.1, L6.2: now also IC1.11 (VDD_PA)
- net at L6.1: now also L4.2, IC1.12 (ANT1); no longer L4.1
- net at L5.1: now also L4.1, IC1.13 (ANT2); no longer L4.2
- net at C16.1: now also IC1.19 (DVDD)
- net at C47.1: now also IC5.19 (DVDD)
- net PB1: now reaches U2.10 (PB1)
- net PB1: now also R11.2, S2.1 (NO_1), S2.2 (NO_2)
- net PB0: now reaches U2.15 (PC3)
- net PB0: now also R9.2, S1.1 (NO_1), S1.2 (NO_2)
- net PB2: now reaches U2.9 (PB2)
- net PB2: now also R17.2, S3.1 (NO_1), S3.2 (NO_2)
- net V-Bat renamed V_Bat
- net V_Bat: now also IC2.6 (V+), R12.2
- new net: IC5.13 (ANT2), L7.1, L9.1
- new net: IC5.12 (ANT1), L7.2, L8.1
- new net: Q2.1 (G), R15.2, R16.1
- new net: Q2.3 (D), Q3.1 (G), R5.1
- new net: C55.2, L9.2
- new net: C49.1, IC5.10 (XC1), R47.1, Y1.3 (CRYSTAL_2)
- new net: C52.1, C54.1, IC5.11 (VDD_PA), L8.2
- new net: IC5.16 (IREF), R6.1
- new net: C48.1, IC5.9 (XC2), R47.2, Y1.1 (CRYSTAL_1)
- new net: LED1.2 (A), R41.1
- new net: IC2.3 (IN+), R12.1, R13.2, R14.2
- new net: IC2.1 (OUT), R14.1, R15.1
- new net: LED3.2 (A), R43.1
- new net: LED2.2 (A), R42.1
- new net: IC2.4 (IN-), IC2.5 (REF)
- new net: LED5.2 (A), R45.1
- new net: LED4.2 (A), R44.1
- new net: LED6.2 (A), R46.1
- new net 50ohm_: C55.1, C56.1
- new net LDO_IN: C12.1, Q3.3 (D), U4.1 (IN), U4.3 (EN)
- no-connect marks 6 -> 36
Other:
- note added: "1 For a charge current of 500ma to battery ISET - Charge Current = 500 mA RISET = KISET / ICHG = 890 / 0.5 = 1780 Ω = 1.8 kΩ standard value 2 Max input current to IC (to prevent excess heat at the HLK-5m05) ILIM - Input Current Cap = 600 mA RILIM = KILIM / IIN-MAX = 1610 / 0.6 = 2683 Ω = 2.7 kΩ standard value"
- note added: "100-240VAC INPUT TO 5V 1A"
- note added: "3V3 LDO"
- note added: "ATtiny1616-S"
- note added: "BQ24074RGT BAT CHARGING SCHEMATICS"
- note added: "COMPARATOR NETWORK FOR LOW BAT SWITCHING"
- note added: "LIGHT SENSING"
- note added: "REMOTE/TRANSMITTER SCHEMATICS"
- note added: "SIX LIGHTING LED ARRAY"
- note added: "STM32G031K8T6TR"
- note added: "SWD TAG CONNECT"
- note added: "USER INPUT BUTTONS"
- note added: "Using a 174 kΩ/100 kΩ divider with a 1 MΩ feedback resistor, I implemented hysteresis in the comparator. This shifts the effective threshold so the circuit turns OFF at ~3.4 V and only turns ON again at ~3.6 V, ensuring clean, stable behavior without oscillation."
- note removed: "1 For a charge current of 500ma ISET - Charge Current = 500 mA RISET = KISET / ICHG = 890 / 0.5 = 1780 Ω = 1.8 kΩ standard value 2 Max input current to IC (to prevent excess heat at the HLK-5m05) ILIM - Input Current Cap = 600 mA RILIM = KILIM / IIN-MAX = 1610 / 0.6 = 2683 Ω = 2.7 kΩ standard value"
- note removed: "Battery voltage sensing"
- moved on the sheet: C1, C10, C11, C12, C14, C16, C19, C2, C21, C22, C23, C25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

Commit message: Update
Parts:
- added D1: LED, LED_SMD:LED_0402_1005Metric, symbol Device:LED
- added H1, H2, H3, H4, H5: MountingHole, MountingHole:MountingHole_3.2mm_M3, symbol Mechanical:MountingHole
- added R52: 330r, Resistor_SMD:R_0402_1005Metric, symbol Device:R
- added TP1: LDO_IN, TestPoint:TestPoint_Pad_D4.0mm, symbol Connector:TestPoint
- added U10, U11, U12, U13, U3, U5, U7, U8, U9: mouse bite, mouse bite:mouse-bite-2mm-4mm, symbol mouse bite:M
- BT1: LCSC Part # (none) -> BC2AAAPC
- C1: JLCPCB PART # C29266 -> (none); LCSC Part # (none) -> C29266
- C10: JLCPCB PART # C125977 -> (none); LCSC Part # (none) -> C2887273
- C11, C5, C8, C9: JLCPCB PART # C98192 -> (none); LCSC Part # (none) -> C98192
- C12: JLCPCB PART # C28323 -> (none); LCSC Part # (none) -> C28323
- C14: JLCPCB PART # C95841 -> (none); LCSC Part # (none) -> C95841
- C16, C47: JLCPCB PART # C106862 -> (none); LCSC Part # (none) -> C106862
- C19: JLCPCB PART # C2918502 -> (none); LCSC Part # (none) -> C2918502
- C2: JLCPCB PART # C94121 -> (none); LCSC Part # (none) -> C94121
- C21, C26, C35, C41: JLCPCB PART # C5440143 -> (none); LCSC Part # (none) -> C5440143
- C22: JLCPCB PART # C18185763 -> (none); LCSC Part # (none) -> C18185763
- C23, C25, C48, C49: JLCPCB PART # C277482 -> (none); LCSC Part # (none) -> C277482
- C28, C50: JLCPCB PART # C76947 -> (none); LCSC Part # (none) -> C76947
- C3, C6, C7: JLCPCB PART # C49678 -> (none); LCSC Part # (none) -> C49678
- C30, C38, C46: JLCPCB PART # C36911349 -> (none); LCSC Part # (none) -> C36911349
- C31, C51: JLCPCB PART # C15195 -> (none); LCSC Part # (none) -> C15195
- C34, C44, C45: JLCPCB PART # C701296 -> (none); LCSC Part # (none) -> C701296
- C36, C53: JLCPCB PART # C60474 -> (none); LCSC Part # (none) -> C60474
- C37: JLCPCB PART # C327009 -> (none); LCSC Part # (none) -> C327009
- C39, C55: JLCPCB PART # C1552 -> (none); LCSC Part # (none) -> C1552
- C4: JLCPCB PART # C46638858 -> (none); LCSC Part # (none) -> C46638858
- C40, C54: JLCPCB PART # C1569 -> (none); LCSC Part # (none) -> C1569
- C42, C56: JLCPCB PART # C710646 -> (none); LCSC Part # (none) -> C710646
- C43, C52: JLCPCB PART # C2987940 -> (none); LCSC Part # (none) -> C2987940
- F1: JLCPCB PART # C136380 -> (none); LCSC Part # (none) -> C136380
- FL2: footprint UU9810MH -> 10MH CHOKE:UU9810MH; JLCPCB PART # C148474 -> (none); LCSC Part # (none) -> C148474
- IC1, IC5: JLCPCB PART # C8791 -> (none); LCSC Part # (none) -> C8791
- IC2: JLCPCB PART # C62505 -> (none); LCSC Part # (none) -> C62505
- IC3: JLCPCB PART # C18164474 -> (none); LCSC Part # (none) -> C18164474
- IC4: JLCPCB PART # C724044 -> (none); LCSC Part # (none) -> C724044
- J1: LCSC Part # (none) -> C160262; now fitted
- J2, J3: now fitted; now in the parts list
- J4, J5, R4: now fitted
- L4, L7: JLCPCB PART # C84404 -> (none); LCSC Part # (none) -> C84404
- L5, L9: JLCPCB PART # C5452416 -> (none); LCSC Part # (none) -> C5452416
- L6, L8: JLCPCB PART # C77108 -> (none); LCSC Part # (none) -> C77108
- LED1, LED2, LED3, LED4, LED5, LED6: JLCPCB PART # 1510-SPMWH1228MD7WATUVKTR-ND -> (none); LCSC Part # (none) -> 1510-SPMWH1228MD7WATUVKTR-ND
- PS1: JLCPCB PART # C209907 -> (none); LCSC Part # (none) -> C209907
- Q1, Q3: JLCPCB PART # C15155 -> (none); LCSC Part # (none) -> C15155; now fitted
- Q2: JLCPCB PART # C20917 -> (none); LCSC Part # (none) -> C20917
- Q4: JLCPCB PART # C20917 -> (none); LCSC Part # (none) -> C20917; now fitted
- R1: JLCPCB PART # C138017 -> (none); LCSC Part # (none) -> C138017
- R10, R13, R29: JLCPCB PART # C60491 -> (none); LCSC Part # (none) -> C60491
- R11, R16, R17, R18, R19, R2, R22, R40, R48, R49, R5, R50, R51, R8, R9: JLCPCB PART # C60490 -> (none); LCSC Part # (none) -> C60490
- R12: JLCPCB PART # C29151471 -> (none); LCSC Part # (none) -> C4214842
- R14, R26, R32, R33, R47: JLCPCB PART # C138033 -> (none); LCSC Part # (none) -> C138033
- R15, R38: JLCPCB PART # C106232 -> (none); LCSC Part # (none) -> C106232
- R20: JLCPCB PART # C125627 -> (none); LCSC Part # (none) -> C125627
- R21, R6: JLCPCB PART # C82868 -> (none); LCSC Part # (none) -> C82868
- R23, R24, R25, R28, R30: JLCPCB PART # C138044 -> (none); LCSC Part # (none) -> C138044
- R27, R35: JLCPCB PART # C137946 -> (none); LCSC Part # (none) -> C137946
- R3: JLCPCB PART # C163481 -> (none); LCSC Part # (none) -> C163481
- R31: JLCPCB PART # C203143 -> (none); LCSC Part # (none) -> C203143
- R34: JLCPCB PART # C482174 -> (none); LCSC Part # (none) -> C482174
- R36: JLCPCB PART # C25760 -> (none); LCSC Part # (none) -> C25760
- R37: JLCPCB PART # C3013173 -> (none); LCSC Part # (none) -> C3013173
- R39: JLCPCB PART # C137976 -> (none); LCSC Part # (none) -> C137976
- R41, R42, R43, R44, R45, R46: footprint Resistor_SMD:R_0402_1005Metric -> Resistor_SMD:R_0805_2012Metric; JLCPCB PART # C138002 -> (none); LCSC Part # (none) -> C2907220
- R7: JLCPCB PART # C105871 -> (none); LCSC Part # (none) -> C105871
- RV1: JLCPCB PART # C2839517 -> (none); LCSC Part # (none) -> C2839517
- S1, S2, S3: JLCPCB PART # C4364459 -> (none); LCSC Part # (none) -> C4364459
- U1: JLCPCB PART # C54313 -> (none); LCSC Part # (none) -> C54313; now fitted
- U2: JLCPCB PART # C614136 -> (none); LCSC Part # (none) -> C614136; now fitted
- U4: JLCPCB PART # C404027 -> (none); LCSC Part # (none) -> C404027; now fitted
- U6: LCSC Part # (none) -> https://www.jotrin.com/product/parts/PIS209S; now fitted
- VR1: JLCPCB PART # C780220 -> (none); LCSC Part # (none) -> C840533
- Y1, Y2: footprint X322516MOB4SI -> crystal:X322516MOB4SI; JLCPCB PART # C12668 -> (none); LCSC Part # (none) -> C12668
Connections:
- net GNDREF: now also D1.1 (K)
- net LDO_IN: now also TP1.1
- net at U2.5 (PA7): now also R52.2
- new net: D1.2 (A), R52.1
- no-connect marks 36 -> 35
Other:
- moved on the sheet: BT1
